Commit message: started new enviornment, using parrot drone

File: install/drone_ignition_bringup/share/drone_ignition_bringup/urdf/common_properties.urdf.xacro (robot description, xacro)
@@ -1,34 +1 @@
-<?xml version="1.0" ?>
-<robot name="xacro_properties" xmlns:xacro="http://ros.org/wiki/xacro">
-  <!-- Init colour -->
-  <material name="black">
-      <color rgba="0.0 0.0 0.0 1.0"/>
-  </material>
-  <material name="dark">
-    <color rgba="0.3 0.3 0.3 1.0"/>
-  </material>
-  <material name="light_black">
-    <color rgba="0.4 0.4 0.4 1.0"/>
-  </material>
-  <material name="blue">
-    <color rgba="0.0 0.0 0.8 1.0"/>
-  </material>
-  <material name="green">
-    <color rgba="0.0 0.8 0.0 1.0"/>
-  </material>
-  <material name="grey">
-    <color rgba="0.5 0.5 0.5 1.0"/>
-  </material>
-  <material name="orange">
-    <color rgba="${255/255} ${108/255} ${10/255} 1.0"/>
-  </material>
-  <material name="brown">
-    <color rgba="${222/255} ${207/255} ${195/255} 1.0"/>
-  </material>
-  <material name="red">
-    <color rgba="0.8 0.0 0.0 1.0"/>
-  </material>
-  <material name="white">
-    <color rgba="1.0 1.0 1.0 1.0"/>
-  </material>
-</robot>
+/home/eleanorlow/robo1/src/drone_ignition_bringup/urdf/common_properties.urdf.xacro

File: install/drone_ignition_bringup/share/drone_ignition_bringup/urdf/drone.gazebo.xacro (robot description, xacro)
@@ -1,172 +1 @@
-<?xml version="1.0"?>
-<robot name="drone" xmlns:xacro="http://ros.org/wiki/xacro">
-  <xacro:arg name="laser_visual"  default="false" />
-  <xacro:arg name="camera_visual" default="false"/>
-  <xacro:arg name="imu_visual"    default="false"/>
-  <xacro:include filename="$(find drone_ignition_bringup)/urdf/proparm.urdf.xacro"/>
-  <gazebo reference="imu_link">
-    <sensor type="imu" name="imu">
-      <always_on>true</always_on>
-      <visualize>$(arg imu_visual)</visualize>
-      <update_rate>100</update_rate>
-      <topic>model/drone/imu</topic>
-      <gz_frame_id>imu_link</gz_frame_id>
-      <imu>
-        <angular_velocity>
-          <x>
-            <noise type="gaussian">
-              <mean>0.0</mean>
-              <stddev>2e-4</stddev>
-              <bias_mean>0.0000075</bias_mean>
-              <bias_stddev>0.0000008</bias_stddev>
-            </noise>
-          </x>
-          <y>
-            <noise type="gaussian">
-              <mean>0.0</mean>
-              <stddev>2e-4</stddev>
-              <bias_mean>0.0000075</bias_mean>
-              <bias_stddev>0.0000008</bias_stddev>
-            </noise>
-          </y>
-          <z>
-            <noise type="gaussian">
-              <mean>0.0</mean>
-              <stddev>2e-4</stddev>
-              <bias_mean>0.0000075</bias_mean>
-              <bias_stddev>0.0000008</bias_stddev>
-            </noise>
-          </z>
-        </angular_velocity>
-        <linear_acceleration>
-          <x>
-            <noise type="gaussian">
-              <mean>0.0</mean>
-              <stddev>1.7e-2</stddev>
-              <bias_mean>0.1</bias_mean>
-              <bias_stddev>0.001</bias_stddev>
-            </noise>
-          </x>
-          <y>
-            <noise type="gaussian">
-              <mean>0.0</mean>
-              <stddev>1.7e-2</stddev>
-              <bias_mean>0.1</bias_mean>
-              <bias_stddev>0.001</bias_stddev>
-            </noise>
-          </y>
-          <z>
-            <noise type="gaussian">
-              <mean>0.0</mean>
-              <stddev>1.7e-2</stddev>
-              <bias_mean>0.1</bias_mean>
-              <bias_stddev>0.001</bias_stddev>
-            </noise>
-          </z>
-        </linear_acceleration>
-      </imu>
-      <plugin
-        filename="ignition-gazebo-imu-system"
-        name="ignition::gazebo::systems::Imu">
-      </plugin>
-    </sensor>
-    <material>Gazebo/Grey</material>
-  </gazebo>
-  <!-- Move base directly without faffing around with diff drive controllers -->
-  <gazebo>
-    <plugin
-      filename="ignition-gazebo-velocity-control-system"
-      name="ignition::gazebo::systems::VelocityControl">
-      <topic>model/drone/cmd_vel</topic>
-    </plugin>
-  </gazebo>
-  <!-- Publish odometry separately -->
-  <gazebo>
-    <plugin
-      filename="ignition-gazebo-odometry-publisher-system"
-      name="ignition::gazebo::systems::OdometryPublisher">
-      <topic>model/drone/odometry</topic>
-      <odom_publish_frequency>20</odom_publish_frequency>
-      <odom_frame>odom</odom_frame>
-      <robot_base_frame>base_link</robot_base_frame>
-    </plugin>
-  </gazebo>
-  <gazebo>
-    <plugin
-      filename="ignition-gazebo-joint-state-publisher-system"
-      name="ignition::gazebo::systems::JointStatePublisher">
-      <topic>model/drone/joint_states</topic>
-    </plugin>
-  </gazebo>
-  <!-- Lidar and cameras use the general Sensors plugin -->
-  <gazebo>
-    <plugin
-        filename="libignition-gazebo-sensors-system.so"
-        name="ignition::gazebo::systems::Sensors">
-    </plugin>
-  </gazebo>
-  <gazebo reference="base_scan">
-    <material>Gazebo/FlatBlack</material>
-    <sensor type="gpu_lidar" name="lidar">
-      <pose relative_to='base_scan'>0 0 0 0 0 0</pose>
-      <visualize>$(arg laser_visual)</visualize>
-      <topic>model/drone/scan</topic>
-      <update_rate>3</update_rate>
-      <gz_frame_id>base_scan</gz_frame_id>
-      <ray>
-        <scan>
-          <horizontal>
-            <samples>360</samples>
-            <resolution>1</resolution>
-            <min_angle>0.0</min_angle>
-            <max_angle>6.28319</max_angle>
-          </horizontal>
-        </scan>
-        <range>
-          <min>0.2</min>
-          <max>40</max>
-          <resolution>0.015</resolution>
-        </range>
-        <noise>
-          <type>gaussian</type>
-          <mean>0.0</mean>
-          <stddev>0.01</stddev>
-        </noise>
-      </ray>
-      <always_on>true</always_on>
-    </sensor>
-  </gazebo>
-  <gazebo reference="camera_link">
-    <sensor name="rgbd_camera" type="rgbd_camera">
-      <camera>
-        <horizontal_fov>2.0944</horizontal_fov>
-        <image>
-          <width>720</width>
-          <height>480</height>
-        </image>
-        <clip>
-          <near>0.1</near>
-          <far>40</far>
-        </clip>
-        <!-- depth_camera near/far clip seems to be ignored for some reason -->
-        <!--    We're using Ignition Gazebo Fortress, which uses sdf format 1.9: http://sdformat.org/tutorials?tut=roadmap -->
-        <!--    This takes the depth_camera parameter with near / far clip http://sdformat.org/spec?ver=1.4&elem=sensor  -->
-        <!-- We also use ign sensors v6 ( run ls | grep libignition-sensors in /usr/lib/x86_64-linux-gnu)-->
-        <!-- Looking at the source code, the sdf sets HasDepthCamera() and corresponding HasDepthNearClip() & HasDepthFarClip() which are used in RgbdCameraSensor.cc, so this should work? -->
-        <!--    SDF description of Camera: https://github.com/gazebosim/sdformat/blob/sdf9/src/Camera.cc#L598-->
-        <!--    Camera sensor source code: https://github.com/gazebosim/gz-sensors/blob/ign-sensors6/src/RgbdCameraSensor.cc#L311  -->
-        <depth_camera>
-          <clip>
-            <near>0.4</near>
-            <far>10</far>
-          </clip>
-        </depth_camera>
-      </camera>
-      <always_on>1</always_on>
-      <update_rate>3</update_rate> <!--10-->
-      <visualize>$(arg camera_visual)</visualize>
-      <topic>/model/drone/camera</topic>
-      <gz_frame_id>camera_link</gz_frame_id>
-    </sensor>
-  </gazebo>
-</robot>
+/home/eleanorlow/robo1/src/drone_ignition_bringup/urdf/drone.gazebo.xacro

File: install/drone_ignition_bringup/share/drone_ignition_bringup/urdf/drone.urdf.xacro (robot description, xacro)
@@ -1,157 +1 @@
-<?xml version="1.0" ?>
-<robot name="drone" xmlns:xacro="http://ros.org/wiki/xacro">
-  <xacro:include filename="$(find drone_ignition_bringup)/urdf/common_properties.urdf.xacro"/>
-  <xacro:include filename="$(find drone_ignition_bringup)/urdf/drone.gazebo.xacro"/>
-  <xacro:include filename="$(find drone_ignition_bringup)/urdf/proparm.urdf.xacro"/>
-  <xacro:property name="r200_cam_rgb_px" value="0.005"/>
-  <xacro:property name="r200_cam_rgb_py" value="0.018"/>
-  <xacro:property name="r200_cam_rgb_pz" value="0.013"/>
-  <xacro:property name="r200_cam_depth_offset" value="0.01"/>
-  <link name="base_link">
-    <visual>
-      <origin xyz="0 0 0.0" rpy="0 -0 0"/>
-      <geometry>
-        <mesh filename="file://$(find drone_ignition_bringup)/urdf/meshes/x4.dae"/>
-      </geometry>
-      <material name="blue"/>
-    </visual>
-    <visual name="base_link_inertia_visual">
-      <origin xyz="0 0 0" rpy="0 -0 0"/>
-      <geometry>
-        <mesh filename="file://$(find drone_ignition_bringup)/urdf/meshes/x4.dae"/>
-      </geometry>
-      <material name="black"/>
-    </visual>
-    <visual name="marker_visual_1">
-      <origin xyz="-0.1 0 0.077" rpy="0 -0.1 0"/>
-      <geometry>
-        <mesh filename="file://$(find drone_ignition_bringup)/urdf/meshes/led.dae" scale= "1 1 1"/>
-      </geometry>
-      <material name="black"/>
-    </visual>
-    <visual name="marker_visual_2">
-      <origin xyz="-0.09 0.059 0.059" rpy="-0.785397 -0 0.2"/>
-      <geometry>
-        <mesh filename="file://$(find drone_ignition_bringup)/urdf/meshes/led.dae" scale= "1 1 1"/>
-      </geometry>
-    </visual>
-    <visual name="marker_visual_3">
-      <origin xyz="-0.09 -0.059 0.059" rpy="0.785397 -0 0.2"/>
-      <geometry>
-        <mesh filename="file://$(find drone_ignition_bringup)/urdf/meshes/led.dae" scale= "1 1 1"/>
-      </geometry>
-      <material name="black"/>
-    </visual>
-    <visual name="downward_flashlight_visual">
-      <origin xyz="-0.043704 0 0.102914" rpy="-0.2 0.000158 -1.57002"/>
-      <geometry>
-        <mesh filename="file://$(find drone_ignition_bringup)/urdf/meshes/spotlight.dae" scale="0.01 0.01 0.01"/>
-      </geometry>
-      <material name="black"/>
-    </visual>
-    <visual name="left_flashlight_visual">
-      <origin xyz="-0.071985 0.090826 0.066102" rpy="0.06 -4.8e-05 -1.27"/>
-      <geometry>
-        <mesh filename="file://$(find drone_ignition_bringup)/urdf/meshes/spotlight.dae" scale="0.01 0.01 0.01"/>
-      </geometry>
-      <material name="black"/>
-    </visual>
-    <visual name="right_flashlight_visual">
-      <origin xyz="-0.071985 -0.090826 0.066102" rpy="0.06 -4.8e-05 -1.87"/>
-      <geometry>
-        <mesh filename="file://$(find drone_ignition_bringup)/urdf/meshes/spotlight.dae" scale="0.01 0.01 0.01"/>
-      </geometry>
-      <material name="black"/>
-    </visual>
-    <collision name="base_link_inertia_collision">
-      <origin xyz="0 0 0" rpy="0 0 0"/>
-      <geometry>
-        <box size="0.3 0.3 0.25"/>
-      </geometry>
-    </collision>
-    <inertial>
-      <origin xyz="0 0 0.062329" rpy="0 0 0"/>
-      <mass value="3.47"/>
-      <inertia ixx="0.075" ixy="-0" ixz="-0"
-               iyy="0.075" iyz="-0"
-               izz="0.148916" />
-    </inertial>
-  </link>
-  <!-- Wheels -->
-  <xacro:wheel wheel_id="front_left" x_pos="0.256" y_pos="${wheel_separation/2}"/>
-  <xacro:wheel wheel_id="front_right" x_pos="0.256" y_pos="-${wheel_separation/2}"/>
-  <xacro:wheel wheel_id="rear_left" x_pos="-0.256" y_pos="${wheel_separation/2}"/>
-  <xacro:wheel wheel_id="rear_right" x_pos="-0.256" y_pos="-${wheel_separation/2}"/>
-  <joint name="imu_joint" type="fixed">
-    <parent link="base_link"/>
-    <child link="imu_link"/>
-    <origin xyz="0.0 0 0.068" rpy="0 0 0"/>
-  </joint>
-  <link name="imu_link"/>
-  <joint name="scan_joint" type="fixed">
-    <parent link="base_link"/>
-    <child link="base_scan"/>
-    <origin xyz="0 0 0.68" rpy="0 0 0"/>
-  </joint>
-  <link name="base_scan">
-    <visual>
-      <origin xyz="0 0 0" rpy="0 0 0"/>
-      <geometry>
-        <cylinder length="0.04" radius="0.09"/>
-      </geometry>
-      <material name="dark"/>
-    </visual>
-    <inertial>
-      <mass value="0" />
-      <origin xyz="0 0 0" />
-      <inertia ixx="0.001" ixy="0.0" ixz="0.0"
-               iyy="0.001" iyz="0.0"
-               izz="0.001" />
-    </inertial>
-  </link>
-  <joint name="camera_joint" type="fixed">
-    <origin xyz="0.45 0.0 0.25" rpy="0 0 0"/> <!-- 0.5 0.0 0.9 -->
-    <parent link="base_link"/>
-    <child link="camera_link"/>
-  </joint>
-  <link name="camera_link">
-    <visual>
-     <origin xyz="0 0 0" rpy="0 0 0"/>
-      <geometry>
-        <box size="0.02 0.08 0.05"/>
-      </geometry>
-      <material name="dark"/>
-    </visual>
-    <visual>
-     <origin xyz="0.015 0 0" rpy="0 1.57 0"/>
-      <geometry>
-        <cylinder length="0.03" radius="0.02"/>
-      </geometry>
-      <material name="dark"/>
-    </visual>
-  </link>
-  <joint name="camera_rgb_joint" type="fixed">
-    <origin xyz="${r200_cam_rgb_px} ${r200_cam_rgb_py} ${r200_cam_rgb_pz}" rpy="0 0 0"/>
-    <parent link="camera_link"/>
-    <child link="camera_rgb_frame"/>
-  </joint>
-  <link name="camera_rgb_frame"/>
-  <joint name="camera_rgb_optical_joint" type="fixed">
-    <origin xyz="0 0 0" rpy="-1.57 0 -1.57"/>
-    <parent link="camera_rgb_frame"/>
-    <child link="camera_rgb_optical_frame"/>
-  </joint>
-  <link name="camera_rgb_optical_frame"/>
-  <joint name="camera_depth_joint" type="fixed">
-    <origin xyz="${r200_cam_rgb_px} ${r200_cam_rgb_py + r200_cam_depth_offset} ${r200_cam_rgb_pz}" rpy="0 0 0"/>
-    <parent link="camera_link"/>
-    <child link="camera_depth_frame"/>
-  </joint>
-  <link name="camera_depth_frame"/>
-  <joint name="camera_depth_optical_joint" type="fixed">
-    <origin xyz="0 0 0" rpy="-1.57 0 -1.57"/>
-    <parent link="camera_depth_frame"/>
-    <child link="camera_depth_optical_frame"/>
-  </joint>
-  <link name="camera_depth_optical_frame"/>
-</robot>
+/home/eleanorlow/robo1/src/drone_ignition_bringup/urdf/drone.urdf.xacro

File: src/drone_ignition_bringup/urdf/drone.gazebo.xacro (robot description, xacro)
@@ -4,5 +4,5 @@
   <xacro:arg name="camera_visual" default="false"/>
   <xacro:arg name="imu_visual"    default="false"/>
-  <xacro:include filename="$(find drone_ignition_bringup)/urdf/proparm.urdf.xacro"/>
+  <!-- <xacro:include filename="$(find 41068_ignition_bringup)/urdf/wheel.urdf.xacro"/> -->
   <gazebo reference="imu_link">
     <sensor type="imu" name="imu">

File: src/drone_ignition_bringup/urdf/drone.urdf.xacro (robot description, xacro)
@@ -3,84 +3,53 @@
   <xacro:include filename="$(find drone_ignition_bringup)/urdf/common_properties.urdf.xacro"/>
   <xacro:include filename="$(find drone_ignition_bringup)/urdf/drone.gazebo.xacro"/>
-  <xacro:include filename="$(find drone_ignition_bringup)/urdf/proparm.urdf.xacro"/>
   <xacro:property name="r200_cam_rgb_px" value="0.005"/>
   <xacro:property name="r200_cam_rgb_py" value="0.018"/>
   <xacro:property name="r200_cam_rgb_pz" value="0.013"/>
   <xacro:property name="r200_cam_depth_offset" value="0.01"/>
+  <!-- Main link -->
   <link name="base_link">
-    <visual>
-      <origin xyz="0 0 0.0" rpy="0 -0 0"/>
+    <inertial>
+      <origin xyz="0 0 0" rpy="0 0 0"/>
+      <mass value="0.503"/> <!-- kg -->
+      <inertia ixx="1.805e-3" ixy="-8.619e-7" ixz="1.555e-5"
+               iyy="1.764e-3" iyz="3.595e-7"
+               izz="3.328e-3" />
+    </inertial>
+<!--     <collision name="collision">
+      <origin xyz="-0.00424 0.00014 -0.00595" rpy="0 0 0"/>
       <geometry>
-        <mesh filename="file://$(find drone_ignition_bringup)/urdf/meshes/x4.dae"/>
+        <box size="0.5 0.5 0.2"/>
       </geometry>
-      <material name="blue"/>
-    </visual>
-    <visual name="base_link_inertia_visual">
-      <origin xyz="0 0 0" rpy="0 -0 0"/>
+    </collision> -->
+    <visual name="hull">
       <geometry>
-        <mesh filename="file://$(find drone_ignition_bringup)/urdf/meshes/x4.dae"/>
-      </geometry>
-      <material name="black"/>
-    </visual>
-    <visual name="marker_visual_1">
-      <origin xyz="-0.1 0 0.077" rpy="0 -0.1 0"/>
-      <geometry>
-        <mesh filename="file://$(find drone_ignition_bringup)/urdf/meshes/led.dae" scale= "1 1 1"/>
-      </geometry>
-      <material name="black"/>
-    </visual>
-    <visual name="marker_visual_2">
-      <origin xyz="-0.09 0.059 0.059" rpy="-0.785397 -0 0.2"/>
-      <geometry>
-        <mesh filename="file://$(find drone_ignition_bringup)/urdf/meshes/led.dae" scale= "1 1 1"/>
+        <mesh filename="file://$(find drone_ignition_bringup)/urdf/meshes/hull.dae"/>
       </geometry>
     </visual>
-    <visual name="marker_visual_3">
-      <origin xyz="-0.09 -0.059 0.059" rpy="0.785397 -0 0.2"/>
+    <visual name="propeller_rr">
+      <origin xyz="-0.09035 -0.11423 -0.00501" rpy="0 0 0"/>
       <geometry>
-        <mesh filename="file://$(find drone_ignition_bringup)/urdf/meshes/led.dae" scale= "1 1 1"/>
+        <mesh filename="file://$(find drone_ignition_bringup)/urdf/meshes/propeller_rr.dae"/>
       </geometry>
-      <material name="black"/>
     </visual>
-    <visual name="downward_flashlight_visual">
-      <origin xyz="-0.043704 0 0.102914" rpy="-0.2 0.000158 -1.57002"/>
+    <visual name="propeller_rl">
+      <origin xyz="0.09035 0.11452 -0.00501" rpy="0 0 0"/>
       <geometry>
-        <mesh filename="file://$(find drone_ignition_bringup)/urdf/meshes/spotlight.dae" scale="0.01 0.01 0.01"/>
+        <mesh filename="file://$(find drone_ignition_bringup)/urdf/meshes/propeller_rl.dae"/>
       </geometry>
-      <material name="black"/>
     </visual>
-    <visual name="left_flashlight_visual">
-      <origin xyz="-0.071985 0.090826 0.066102" rpy="0.06 -4.8e-05 -1.27"/>
+    <visual name="propeller_fr">
+      <origin xyz="0.08456 -0.11435 -0.00501" rpy="0 0 0"/>
       <geometry>
-        <mesh filename="file://$(find drone_ignition_bringup)/urdf/meshes/spotlight.dae" scale="0.01 0.01 0.01"/>
+        <mesh filename="file://$(find drone_ignition_bringup)/urdf/meshes/propeller_fr.dae"/>
       </geometry>
-      <material name="black"/>
     </visual>
-    <visual name="right_flashlight_visual">
-      <origin xyz="-0.071985 -0.090826 0.066102" rpy="0.06 -4.8e-05 -1.87"/>
+    <visual name="propeller_fl">
+      <origin xyz="0.08456 0.11463 -0.00501" rpy="0 0 0"/>
       <geometry>
-        <mesh filename="file://$(find drone_ignition_bringup)/urdf/meshes/spotlight.dae" scale="0.01 0.01 0.01"/>
+        <mesh filename="file://$(find drone_ignition_bringup)/urdf/meshes/propeller_fl.dae"/>
       </geometry>
-      <material name="black"/>
     </visual>
-    <collision name="base_link_inertia_collision">
-      <origin xyz="0 0 0" rpy="0 0 0"/>
-      <geometry>
-        <box size="0.3 0.3 0.25"/>
-      </geometry>
-    </collision>
-    <inertial>
-      <origin xyz="0 0 0.062329" rpy="0 0 0"/>
-      <mass value="3.47"/>
-      <inertia ixx="0.075" ixy="-0" ixz="-0"
-               iyy="0.075" iyz="-0"
-               izz="0.148916" />
-    </inertial>
   </link>
-  <!-- Wheels -->
-  <xacro:wheel wheel_id="front_left" x_pos="0.256" y_pos="${wheel_separation/2}"/>
-  <xacro:wheel wheel_id="front_right" x_pos="0.256" y_pos="-${wheel_separation/2}"/>
-  <xacro:wheel wheel_id="rear_left" x_pos="-0.256" y_pos="${wheel_separation/2}"/>
-  <xacro:wheel wheel_id="rear_right" x_pos="-0.256" y_pos="-${wheel_separation/2}"/>
   <joint name="imu_joint" type="fixed">
     <parent link="base_link"/>
@@ -92,5 +61,5 @@
     <parent link="base_link"/>
     <child link="base_scan"/>
-    <origin xyz="0 0 0.68" rpy="0 0 0"/>
+    <origin xyz="0 0 0.2" rpy="0 0 0"/>
   </joint>
   <link name="base_scan">
@@ -111,5 +80,5 @@
   </link>
   <joint name="camera_joint" type="fixed">
-    <origin xyz="0.45 0.0 0.25" rpy="0 0 0"/> <!-- 0.5 0.0 0.9 -->
+    <origin xyz="0.25 0.0 0.25" rpy="0 0.785398 0"/> <!-- 0.5 0.0 0.9 -->
     <parent link="base_link"/>
     <child link="camera_link"/>
