Commit message: first edit of gazebo worlds

File: src/drone_ignition_bringup/urdf/common_properties.urdf.xacro (robot description, xacro)
@@ -2,5 +2,5 @@
 <robot name="xacro_properties" xmlns:xacro="http://ros.org/wiki/xacro">
   <!-- Init colour -->
-  <material name="black">
+  <material name="purple">
       <color rgba="0.0 0.0 0.0 1.0"/>
   </material>
